Commit message: add platform trajectory file

File: workspace/src/platform_description/urdf/husky.urdf (robot description, URDF)
Before this commit: robot husky, 15 links, 14 joints
Links:
- link front_bumper_link: geometry visual mesh filename=package://platform_description/meshes/bumper.dae
- link front_left_wheel_link: geometry collision cylinder length=0.1143 radius=0.1651; visual mesh filename=package://platform_description/meshes/wheel.dae
- link front_right_wheel_link: geometry collision cylinder length=0.1143 radius=0.1651; visual mesh filename=package://platform_description/meshes/wheel.dae
- link rear_bumper_link: geometry visual mesh filename=package://platform_description/meshes/bumper.dae
- link rear_left_wheel_link: geometry collision cylinder length=0.1143 radius=0.1651; visual mesh filename=package://platform_description/meshes/wheel.dae
- link rear_right_wheel_link: geometry collision cylinder length=0.1143 radius=0.1651; visual mesh filename=package://platform_description/meshes/wheel.dae
- link top_chassis_link: geometry visual mesh filename=package://platform_description/meshes/top_chassis.dae
- link top_plate_link: geometry collision mesh filename=package://platform_description/meshes/top_plate.stl scale=3 3 0.001; visual mesh filename=package://platform_description/meshes/top_plate.dae scale=3 3 0.001
- link user_rail_link: geometry visual mesh filename=package://platform_description/meshes/user_rail.dae

Commit message: Update README.md

File: workspace/src/platform_description/urdf/husky.urdf (robot description, URDF)
Before this commit: robot husky, 15 links, 14 joints
Links:
- link top_plate_link: geometry collision mesh filename=package://platform_description/meshes/top_plate.stl scale=3 2 0.001; visual mesh filename=package://platform_description/meshes/top_plate.dae scale=3 2 0.001
